Commit message: multiple robots in gazebo

File: src/diff_drive_robot/urdf/robot.gazebo.xacro (robot description, xacro)
@@ -1,32 +1,30 @@
 <?xml version="1.0"?>
-<robot>
-    <!-- Differential drive plugin -->
+<robot xmlns:xacro="http://www.ros.org/wiki/xacro">
+    <xacro:arg name="ns" default="r0"/>
     <gazebo>
         <plugin filename="gz-sim-diff-drive-system" name="gz::sim::systems::DiffDrive">
-            <right_joint>right_wheel_joint</right_joint>
-            <left_joint>left_wheel_joint</left_joint>
+            <right_joint>$(arg ns)/right_wheel_joint</right_joint>
+            <left_joint>$(arg ns)/left_wheel_joint</left_joint>
             <wheel_separation>0.35</wheel_separation>
             <wheel_radius>0.05</wheel_radius>
             <max_linear_acceleration>10</max_linear_acceleration>
-            <topic>cmd_vel</topic>
+            <topic>$(arg ns)/cmd_vel</topic>
         </plugin>
-        <!-- Odometry publisher -->
         <plugin filename="gz-sim-odometry-publisher-system" name="gz::sim::systems::OdometryPublisher">
-            <odom_frame>odom</odom_frame>
-            <robot_base_frame>base_link</robot_base_frame>
+            <odom_frame>$(arg ns)/odom</odom_frame>
+            <robot_base_frame>$(arg ns)/base_link</robot_base_frame>
             <odom_publish_frequency>50</odom_publish_frequency>
-            <odom_topic>/odom</odom_topic>
-            <tf_topic>/tf</tf_topic>
+            <odom_topic>$(arg ns)/odom</odom_topic>
+            <tf_topic>$(arg ns)/tf</tf_topic>
             <dimensions>2</dimensions>
         </plugin>
-        <!-- Joint state publisher -->
         <plugin filename="gz-sim-joint-state-publisher-system" name="gz::sim::systems::JointStatePublisher">
-            <topic>joint_states</topic>
-            <joint_name>right_wheel_joint</joint_name>
-            <joint_name>left_wheel_joint</joint_name>
+            <topic>$(arg ns)/joint_states</topic>
+            <joint_name>$(arg ns)/right_wheel_joint</joint_name>
+            <joint_name>$(arg ns)/left_wheel_joint</joint_name>
         </plugin>
     </gazebo>
     <!-- LiDAR (PointCloud2) -->
-    <gazebo reference="laser_frame">
+    <gazebo reference="$(arg ns)/laser_frame">
         <sensor type="gpu_ray" name="lidar_sensor">
             <pose>0 0 0 0 0 0</pose>
@@ -60,6 +58,6 @@
                 <output_type>point_cloud</output_type>
             </ray>
-            <topic>pointcloud</topic>
-            <frame_name>laser_frame</frame_name>
+            <topic>$(arg ns)/pointcloud</topic>
+            <frame_name>$(arg ns)/laser_frame</frame_name>
         </sensor>
     </gazebo>

File: src/diff_drive_robot/urdf/robot.xacro (robot description, xacro)
@@ -1,16 +1,17 @@
 <?xml version="1.0"?>
-<robot name="diff_drive_robot" xmlns:xacro="http://www.ros.org/wiki/xacro" >
-    <xacro:include filename="$(find diff_drive_robot)/urdf/robot.gazebo" />
+<robot name="diff_drive_robot" xmlns:xacro="http://www.ros.org/wiki/xacro">
+    <xacro:arg name="ns" default="r0"/>
     <xacro:include filename="inertial_macros.xacro" />
+    <xacro:include filename="robot.gazebo.xacro" />
     <!-- Base link -->
-    <link name="base_link">
+    <link name="$(arg ns)/base_link">
     </link>
     <!-- Chassis link -->
-    <joint name="chassis_joint" type="fixed">
-        <parent link="base_link"/>
-        <child link="chassis"/>
+    <joint name="$(arg ns)/chassis_joint" type="fixed">
+        <parent link="$(arg ns)/base_link"/>
+        <child link="$(arg ns)/chassis"/>
         <origin xyz="-0.1 0 0"/>
     </joint>
-    <link name="chassis">
+    <link name="$(arg ns)/chassis">
         <visual>
             <origin xyz="0.15 0 0.075"/>
@@ -33,11 +34,11 @@
     </link>
     <!-- Left wheel -->
-    <joint name="left_wheel_joint" type="continuous">
+    <joint name="$(arg ns)/left_wheel_joint" type="continuous">
         <origin xyz="0 0.175 0" rpy="-${pi/2} 0 0"/>
-        <child link="left_wheel"/>
-        <parent link="base_link"/>
+        <child link="$(arg ns)/left_wheel"/>
+        <parent link="$(arg ns)/base_link"/>
         <axis xyz="0 0 1"/>
     </joint>
-    <link name="left_wheel">
+    <link name="$(arg ns)/left_wheel">
         <xacro:inertial_cylinder mass="0.1" length="0.04" radius="0.05">
             <origin xyz="0 0 0" rpy="0 0 0"/>
@@ -58,11 +59,11 @@
     </link>
     <!-- Right wheel -->
-    <joint name="right_wheel_joint" type="continuous">
+    <joint name="$(arg ns)/right_wheel_joint" type="continuous">
         <origin xyz="0 -0.175 0" rpy="${pi/2} 0 0"/>
-        <child link="right_wheel"/>
-        <parent link="base_link"/>
+        <child link="$(arg ns)/right_wheel"/>
+        <parent link="$(arg ns)/base_link"/>
         <axis xyz="0 0 -1"/>
     </joint>
-    <link name="right_wheel">
+    <link name="$(arg ns)/right_wheel">
         <xacro:inertial_cylinder mass="0.1" length="0.04" radius="0.05">
             <origin xyz="0 0 0" rpy="0 0 0"/>
@@ -83,10 +84,10 @@
     </link>
     <!-- Castor wheel -->
-    <joint name="castor_wheel_joint" type="fixed">
-        <parent link="chassis"/>
-        <child link="castor_wheel"/>
+    <joint name="$(arg ns)/castor_wheel_joint" type="fixed">
+        <parent link="$(arg ns)/chassis"/>
+        <child link="$(arg ns)/castor_wheel"/>
         <origin xyz="0.24 0 0"/>
     </joint>
-    <link name="castor_wheel">
+    <link name="$(arg ns)/castor_wheel">
         <xacro:inertial_sphere mass="0.4" radius="0.05">
             <origin xyz="0 0 0" rpy="0 0 0"/>
@@ -107,27 +108,27 @@
     </link>
     <!-- Gazebo friction parameters -->
-    <gazebo reference="left_wheel">
+    <gazebo reference="$(arg ns)/left_wheel">
         <mu1>1.0</mu1>
         <mu2>1.0</mu2>
     </gazebo>
-    <gazebo reference="right_wheel">
+    <gazebo reference="$(arg ns)/right_wheel">
         <mu1>1.0</mu1>
         <mu2>1.0</mu2>
     </gazebo>
-    <gazebo reference="castor_wheel">
+    <gazebo reference="$(arg ns)/castor_wheel">
         <mu1>0.000001</mu1>
         <mu2>0.000001</mu2>
     </gazebo>
-    <gazebo reference="base_link">
+    <gazebo reference="$(arg ns)/base_link">
         <mu1>1.0</mu1>
         <mu2>1.0</mu2>
     </gazebo>
     <!-- Lidar link (visual only) -->
-    <joint name="laser_joint" type="fixed">
-        <parent link="chassis"/>
-        <child link="laser_frame"/>
+    <joint name="$(arg ns)/laser_joint" type="fixed">
+        <parent link="$(arg ns)/chassis"/>
+        <child link="$(arg ns)/laser_frame"/>
         <origin xyz="0.1 0 0.175" rpy="0 0 0"/>
     </joint>
-    <link name="laser_frame">
+    <link name="$(arg ns)/laser_frame">
         <visual>
             <origin xyz="0 0 0"/>
